File: pcb/rev3/GEA-Adapter-Rev3.kicad_pcb (KiCad board)
At the start: 2 copper layers, 72 x 34 mm, 88 parts, among them J1 8P8C, J3 TC2030, J4 USB_C_Receptacle_USB2.0_16P, Q1 Si2309CDS, Q2 Si2309CDS, SW1 SW_Push, SW2 SW_Push, U2 ESP32-C3-WROOM-02, U4 74LVC2G07, U5 74LVC2G07_3v3, U6 AP2112K-3.3, U7 USBLC6-2SC6, U8 AP63205WU

Commit message: feat(pcb): route rev3a GEA3 MCU paths
Routing:
- net GEA3_RX: track 0.00 -> 40.1 mm, vias 0 -> 2
- net GEA3_TX: track 0.00 -> 34.1 mm, vias 0 -> 2
Changed lines of the file:
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@@
+	)
+	(segment
+		(start 24.5 18.9125)
+		(end 25.6 20)
+		(width 0.25)
+		(layer "F.Cu")
+		(net 28)
+	)
+	(segment
+		(start 55.9 25.75)
+		(end 55.9 27)
+		(width 0.25)
+		(layer "F.Cu")
+		(net 28)
+	)
+	(via
+		(at 55.9 27)
+		(size 0.6)
+		(drill 0.3)
+		(layers "F.Cu" "B.Cu")
+		(net 28)
+	)
+	(via
+		(at 25.6 20)
+		(size 0.6)
+		(drill 0.3)
+		(layers "F.Cu" "B.Cu")
+		(net 28)
+	)
+	(segment
+		(start 25.6 20)
+		(end 55.9 20)
+		(width 0.25)
+		(layer "B.Cu")
+		(net 28)
+	)
+	(segment
+		(start 55.9 20)
+		(end 55.9 27)
+		(width 0.25)
+		(layer "B.Cu")
+		(net 28)
+	)
+	(segment
+		(start 54.4 25.75)
+		(end 54.4 27)
+		(width 0.25)
+		(layer "F.Cu")
+		(net 29)
+	)
+	(segment
+		(start 28.9 18.9125)
+		(end 29 20.1)
+		(width 0.25)
+		(layer "F.Cu")
+		(net 29)
+	)
+	(segment
+		(start 29 20.1)
+		(end 31.8 20.8)
+		(width 0.25)
+		(layer "F.Cu")
+		(net 29)
+	)
+	(via
+		(at 54.4 27)
+		(size 0.6)
+		(drill 0.3)
+		(layers "F.Cu" "B.Cu")
+		(net 29)
+	)
+	(via
+		(at 31.8 20.8)
+		(size 0.6)
+		(drill 0.3)
+		(layers "F.Cu" "B.Cu")
+		(net 29)
+	)
+	(segment
+		(start 31.8 20.8)
+		(end 31.8 21.4)
+		(width 0.25)
+		(layer "B.Cu")
+		(net 29)
+	)
+	(segment
+		(start 31.8 21.4)
+		(end 54.4 21.4)
+		(width 0.25)
+		(layer "B.Cu")
+		(net 29)
+	)
+	(segment
+		(start 54.4 21.4)
+		(end 54.4 27)
+		(width 0.25)
+		(layer "B.Cu")
+		(net 29)
 	)
 	(segment

Commit message: feat(pcb): route rev3a local 3v3 branches
Routing:
- net +3V3: track 5.79 -> 15.3 mm
Changed lines of the file:
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@@
+	)
+	(segment
+		(start 52.5 4.0875)
+		(end 55 5.9125)
+		(width 0.5)
+		(layer "F.Cu")
+		(net 1)
 	)
 	(segment
 		(start 64.9 8.25)
 		(end 64.9 5.3)
+		(width 0.5)
+		(layer "F.Cu")
+		(net 1)
+	)
+	(segment
+		(start 47.5 10.55)
+		(end 50.5 13.45)
 		(width 0.5)
 		(layer "F.Cu")
@@
 		(width 0.5)
 		(layer "F.Cu")
+		(net 1)
+	)
+	(segment
+		(start 56.95 29)
+		(end 59 28.0875)
+		(width 0.5)
+		(layer "F.Cu")

Commit message: feat(pcb): route rev3a 3v3 control island
Routing:
- net +3V3: track 15.3 -> 31.9 mm, vias 0 -> 3
Changed lines of the file:
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@@
+	)
+	(segment
+		(start 31.1 18.9125)
+		(end 32 18.2)
+		(width 0.5)
+		(layer "F.Cu")
+		(net 1)
 	)
 	(segment
 		(start 64.9 8.25)
 		(end 64.9 5.3)
+		(width 0.5)
+		(layer "F.Cu")
+		(net 1)
+	)
+	(segment
+		(start 26.7 15.1125)
+		(end 27.5 14.5)
 		(width 0.5)
 		(layer "F.Cu")
@@
 		(start 64.9 5.3)
 		(end 64.75 5.3)
+		(width 0.5)
+		(layer "F.Cu")
+		(net 1)
+	)
+	(segment
+		(start 26.7 18.9125)
+		(end 27.5 19.1)
 		(width 0.5)
 		(layer "F.Cu")
@@
 		(net 1)
 	)
+	(via
+		(at 27.5 19.1)
+		(size 0.8)
+		(drill 0.4)
+		(layers "F.Cu" "B.Cu")
+		(net 1)
+	)
+	(via
+		(at 27.5 14.5)
+		(size 0.8)
+		(drill 0.4)
+		(layers "F.Cu" "B.Cu")
+		(net 1)
+	)
+	(via
+		(at 32 18.2)
+		(size 0.8)
+		(drill 0.4)
+		(layers "F.Cu" "B.Cu")
+		(net 1)
+	)
+	(segment
+		(start 27.5 19.1)
+		(end 32 19.1)
+		(width 0.5)
+		(layer "B.Cu")
+		(net 1)
+	)
+	(segment
+		(start 32 19.1)
+		(end 32 18.2)
+		(width 0.5)
+		(layer "B.Cu")
+		(net 1)
+	)
+	(segment
+		(start 27.5 14.5)
+		(end 32 14.5)
+		(width 0.5)
+		(layer "B.Cu")
+		(net 1)
+	)
+	(segment
+		(start 32 14.5)
+		(end 32 18.2)
+		(width 0.5)
+		(layer "B.Cu")
+		(net 1)
+	)

Commit message: feat(pcb): route rev3a reset and led control nets
Routing:
- net /EN: track 0.00 -> 12.1 mm, vias 0 -> 2
- net /LED2: track 0.00 -> 6.64 mm
Changed lines of the file:
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@@
+	)
+	(segment
+		(start 57.0875 5)
+		(end 56.5 5)
+		(width 0.25)
+		(layer "F.Cu")
+		(net 11)
+	)
+	(segment
+		(start 63.4 7.4)
+		(end 63.4 8.25)
+		(width 0.25)
+		(layer "F.Cu")
+		(net 11)
+	)
+	(segment
+		(start 56.5 5)
+		(end 56.5 6.2)
+		(width 0.25)
+		(layer "F.Cu")
+		(net 11)
+	)
+	(via
+		(at 56.5 6.2)
+		(size 0.8)
+		(drill 0.4)
+		(layers "F.Cu" "B.Cu")
+		(net 11)
+	)
+	(via
+		(at 63.4 7.4)
+		(size 0.8)
+		(drill 0.4)
+		(layers "F.Cu" "B.Cu")
+		(net 11)
+	)
+	(segment
+		(start 62.5 7.4)
+		(end 63.4 7.4)
+		(width 0.25)
+		(layer "B.Cu")
+		(net 11)
+	)
+	(segment
+		(start 62.5 5.5)
+		(end 62.5 7.4)
+		(width 0.25)
+		(layer "B.Cu")
+		(net 11)
+	)
+	(segment
+		(start 56.5 6.2)
+		(end 56.5 5.5)
+		(width 0.25)
+		(layer "B.Cu")
+		(net 11)
+	)
+	(segment
+		(start 56.5 5.5)
+		(end 62.5 5.5)
+		(width 0.25)
+		(layer "B.Cu")
+		(net 11)
+	)
+	(segment
+		(start 61.5 30.6)
+		(end 61.5 29.9125)
+		(width 0.25)
+		(layer "F.Cu")
+		(net 13)
+	)
+	(segment
+		(start 60.4 25.75)
+		(end 60.4 30.6)
+		(width 0.25)
+		(layer "F.Cu")
+		(net 13)
+	)
+	(segment
+		(start 60.4 30.6)
+		(end 61.5 30.6)
+		(width 0.25)
+		(layer "F.Cu")
+		(net 13)
 	)
 	(segment

Commit message: feat(pcb): route rev3a boot and debug-led escapes
Routing:
- net /DBG_LED: track 0.00 -> 9.20 mm, vias 0 -> 2
- net /BOOT: track 0.00 -> 5.85 mm, vias 0 -> 2
Changed lines of the file:
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@@
+	)
+	(segment
+		(start 55 4.0875)
+		(end 55.8 3.6)
+		(width 0.25)
+		(layer "F.Cu")
+		(net 5)
+	)
+	(segment
+		(start 54.4 7.2)
+		(end 54.4 8.25)
+		(width 0.25)
+		(layer "F.Cu")
+		(net 5)
+	)
+	(via
+		(at 54.4 7.2)
+		(size 0.8)
+		(drill 0.4)
+		(layers "F.Cu" "B.Cu")
+		(net 5)
+	)
+	(via
+		(at 55.8 3.6)
+		(size 0.8)
+		(drill 0.4)
+		(layers "F.Cu" "B.Cu")
+		(net 5)
+	)
+	(segment
+		(start 55.8 3.6)
+		(end 54.4 7.2)
+		(width 0.25)
+		(layer "B.Cu")
+		(net 5)
 	)
 	(segment
@@
 	)
 	(segment
+		(start 61.9 25.75)
+		(end 62.5 26.8)
+		(width 0.25)
+		(layer "F.Cu")
+		(net 10)
+	)
+	(segment
+		(start 59 30.6)
+		(end 59 29.9125)
+		(width 0.25)
+		(layer "F.Cu")
+		(net 10)
+	)
+	(via
+		(at 62.5 26.8)
+		(size 0.6)
+		(drill 0.3)
+		(layers "F.Cu" "B.Cu")
+		(net 10)
+	)
+	(via
+		(at 59 30.6)
+		(size 0.6)
+		(drill 0.3)
+		(layers "F.Cu" "B.Cu")
+		(net 10)
+	)
+	(segment
+		(start 62.5 30.6)
+		(end 59 30.6)
+		(width 0.25)
+		(layer "B.Cu")
+		(net 10)
+	)
+	(segment
+		(start 62.5 26.8)
+		(end 62.5 30.6)
+		(width 0.25)
+		(layer "B.Cu")
+		(net 10)
+	)
+	(segment

Commit message: feat(pcb): route rev3a button terminal pairs
Routing:
- net /BOOT_SEL: track 0.00 -> 6.00 mm
- net /BOOT: track 5.85 -> 11.8 mm
Changed lines of the file:
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@@
+		(net 5)
+	)
+	(segment
+		(start 10 5.275)
+		(end 16 5.275)
+		(width 0.25)
+		(layer "F.Cu")
 		(net 5)
 	)
@@
 	)
 	(segment
+		(start 2 1.525)
+		(end 8 1.525)
+		(width 0.25)
+		(layer "F.Cu")
+		(net 6)
+	)
+	(segment

Commit message: feat(pcb): route rev3a protection and led branches
Routing:
- net Net-(D5-A): track 0.00 -> 8.11 mm
- net Net-(D9-A): track 0.00 -> 2.86 mm
- net Net-(R20-Pad1): track 0.00 -> 2.20 mm
Changed lines of the file:
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@@
+	)
+	(segment
+		(start 7.3 6.2)
+		(end 12.7 6.2)
+		(width 0.25)
+		(layer "F.Cu")
+		(net 35)
+	)
+	(segment
+		(start 12.7 6.2)
+		(end 13.0875 7.5)
+		(width 0.25)
+		(layer "F.Cu")
+		(net 35)
+	)
+	(segment
+		(start 6.9375 7.5)
+		(end 7.3 6.2)
+		(width 0.25)
+		(layer "F.Cu")
+		(net 35)
+	)
+	(segment
+		(start 30.5 21.6875)
+		(end 32.7 23.5125)
+		(width 0.25)
+		(layer "F.Cu")
+		(net 37)
 	)
 	(segment
@@
 	)
 	(segment
+		(start 35.8 19.9125)
+		(end 38 19.9125)
+		(width 0.25)
+		(layer "F.Cu")
+		(net 47)
+	)
+	(segment

Commit message: feat(pcb): connect rev3a buffer ground returns
Routing:
- net GND: track 51.4 -> 53.5 mm, vias 8 -> 10
Changed lines of the file:
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@@
+	)
+	(segment
+		(start 19.8625 19)
+		(end 18.8 19)
+		(width 0.25)
+		(layer "F.Cu")
+		(net 33)
 	)
 	(segment
@@
 		(end 37.675 27.65)
 		(width 0.5)
+		(layer "F.Cu")
+		(net 33)
+	)
+	(segment
+		(start 20.5 21.6875)
+		(end 19.5 21.6875)
+		(width 0.25)
 		(layer "F.Cu")
 		(net 33)
@@
 		(layers "F.Cu" "B.Cu")
 		(net 33)
+	)
+	(via
+		(at 19.5 21.6875)
+		(size 0.6)
+		(drill 0.3)
+		(layers "F.Cu" "B.Cu")
+		(net 33)
+	)
+	(via
+		(at 18.8 19)
+		(size 0.6)
+		(drill 0.3)
+		(layers "F.Cu" "B.Cu")
+		(net 33)
