File: pcb/rev3/GEA-Adapter-Rev3.kicad_sch (KiCad schematic)
At the start: 110 parts, among them J1 8P8C, J2 1x6, J3 TC2030, J4 USB_C_Receptacle_USB2.0_16P, Q3 CJ3407, Q4 CJ3407, Q5 MMBT3904, SW1 SW_Push, SW2 SW_Push, U10 TPS22810DBVR, U2 ESP32-C3-WROOM-02, U4 74LVC2G07, U5 74LVC2G07_3v3, U6 AP2112K-3.3, U7 USBLC6-2SC6, U8 AP63205WU, U9 TPS22810DBVR

Commit message: docs(pcb): prepare rev3a schematic review
Parts:
- D4: MPN (none) -> KT-0805G; Manufacturer (none) -> Hubei KENTO Elec
- D5: MPN (none) -> NCD0805R1; Manufacturer (none) -> Foshan NationStar Optoelectronics
- D6: MPN (none) -> KT-0805Y; Manufacturer (none) -> Hubei KENTO Elec
Other:
- note added: "1 APPLIANCE CONNECTOR / PROTECTED INPUTS"
- note added: "2 POWER COMBINING -> AP63205 / NOMINAL +5V"
- note added: "3 3.3V REGULATOR"
- note added: "4 ESP32-C3 / UART"
- note added: "5 USB-C / ESD / USB DATA"
- note added: "DESIGN REVIEW NOTES Pin 1 has priority when both appliance inputs are present; blocking diodes prevent cross-feed. AP63205 output is nominal +5V and requires source headroom; validate all eight source states current-limited. USB-C VBUS is isolated from appliance input; verify enumeration and no backfeed on prototype. U9/U10 QOD pin 5: NC. DNP/exclude states and source metadata are retained."
- note removed: "2.1 changes Added ground test point Change D8 to bigger part move rj45 inboard 4.5mm smaller 7805 or different ldo"
- note removed: "DIAGNOSTIC TEST PADS Optional top-side SMD pads for bring-up"
- note removed: "Decoupling Caps"
- note removed: "Dryer Only 1, 7 & 8 populated with pins Washer Only 1, 3,4,5,6,8 populated with pins"
- note removed: "ESD Protection"
- note removed: "MOSFET GATE PROTECTION 12 V DC clamps; ESD/EFT unresolved"
- note removed: "NATIVE USB-C (USB 2.0 DEVICE + ISOLATED 5 V INPUT)"
- note removed: "Peak of 1.5 amps w/o inrush"
- note removed: "REV 3A WIDE-INPUT BUCK + ISOLATED 5 V POWER"
- note removed: "Reverse polarity protection and inrush current limit"
- note removed: "T-568B Brn Brn/Wht Grn Blu/Wht Blu Grn/Wht Orn Orn/Wht"
- note removed: "Tried to be compatible with FirstBuild v1.0 DBG Led ~inverted~ GPIO9 is strapping pin. Pull down by GEA bus could be a problem. JP1 defaults to GPIO5"
- note removed: "VDC +9v to +16v"
- note removed: "Voltage Supervisor, Hold ESP reset for 150ms after power reaches 2.9V. Prevent brownout at boot."
- note removed: "Washer Blk NC Grn/Rd Org BLU BRN NC RED"
- note removed: "Washer GND NC Hvoltage side RX/TX RX/TX +5V NC +16.2V"
- title: GEA Adapter -> GE Appliance Adapter - Rev3A
- moved on the sheet: D10, F3, J4, R26, R27, R28, R29, U7
