File: pcb/rev3/GEA-Adapter-Rev3.kicad_sch (KiCad schematic)
At the start: 110 parts, among them J1 8P8C, J2 1x6, J3 TC2030, J4 USB_C_Receptacle_USB2.0_16P, Q3 CJ3407, Q4 CJ3407, Q5 MMBT3904, SW1 SW_Push, SW2 SW_Push, U10 TPS22810DBVR, U2 ESP32-C3-WROOM-02, U4 74LVC2G07, U5 74LVC2G07_3v3, U6 AP2112K-3.3, U7 USBLC6-2SC6, U8 AP63205WU, U9 TPS22810DBVR

Commit message: docs(pcb): prepare rev3a schematic review
Parts:
- Q3, Q4: symbol Device:Q_PMOS_GSD -> Transistor_FET:Q_PMOS_GSD
Other:
- moved on the sheet: C10, C11, C12, C13, C14, C15, C16, C17, C18, C20, C21, C22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

Commit message: fix(pcb): use assembly-ready usb-c connector
Parts:
- J4: LCSC C2894897 -> C2765186; MPN HC-TYPE-C-16P-01A -> TYPE-C 16PIN 2MD(073); Manufacturer HCTL -> SHOU HAN
Changed lines of the file:
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@@
 			)
 		)
-		(property "Datasheet" "https://datasheet.lcsc.com/datasheet/pdf/7d87e82d7c94fc2f1ad4584993e52b86.pdf?productCode=C2894897"
+		(property "Datasheet" "https://jlcpcb.com/partdetail/C2765186"
 			(at 413.81 185 0)
 			(hide yes)
@@
 			)
 		)
-		(property "Description" "HCTL USB 2.0 Type-C receptacle, 16 contacts, top mount"
+		(property "Description" "SHOU HAN USB 2.0 Type-C receptacle, 16 contacts, top mount"
 			(at 410 185 0)
 			(hide yes)
@@
 			)
 		)
-		(property "Manufacturer" "HCTL"
+		(property "Manufacturer" "SHOU HAN"
 			(at 410 185 0)
 			(effects
@@
 			)
 		)
-		(property "MPN" "HC-TYPE-C-16P-01A"
+		(property "MPN" "TYPE-C 16PIN 2MD(073)"
 			(at 410 185 0)
 			(effects
@@
 			)
 		)
-		(property "LCSC" "C2894897"
+		(property "LCSC" "C2765186"
 			(at 410 185 0)
 			(effects

Commit message: feat(pcb): improve rev3a recovery and review artifacts
Connections:
- net BOOT_SEL: no longer SW1.1
- net EN: now also SW1.1
Changed lines of the file:
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@@
-	(wire
-		(pts
-			(xy 161.29 160.02) (xy 161.29 182.88)
-		)
-		(stroke
-			(width 0)
-			(type default)
-		)
-	)
 	(wire
 		(pts
@@
 	(label "BOOT_SEL"
 		(at 151.13 160.02 0)
+		(effects
+			(font
+				(size 1.27 1.27)
+			)
+			(justify left bottom)
+		)
+	)
+	(label "EN"
+		(at 161.29 182.88 0)
 		(effects
 			(font
@@
 			)
 		)
-		(property "Description" "DNP Tag-Connect TC2030 programming footprint; pads present on PCB; do not install cable during normal operation"
+		(property "Description" "DNP connector-free Tag-Connect recovery footprint; manual flash fallback when USB is unavailable; no installed part"
 			(at 49.53 232.41 0)
 			(effects

Commit message: fix(pcb): finalize rev3a sourcing and connector model
Parts:
- C1, C12, C14, C24, C25, C3, C4, C5, C6, C7: LCSC C28233 -> C106243; MPN CL21B104KCFNNNE -> CC0805KKX7R0BB104; Manufacturer Samsung Electro-Mechanics -> Yageo
- C2, C20, C21: LCSC C28323 -> C91185; MPN CL21B105KBFNNNE -> CC0805KKX7R9BB105; Manufacturer Samsung -> Yageo
Changed lines of the file:
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@@
 			)
 		)
-		(property "Description" "C28233"
+		(property "Description" "C106243"
 			(at 36.83 140.97 0)
 			(effects
@@
 			)
 		)
-		(property "LCSC" "C28233"
+		(property "LCSC" "C106243"
 			(at 36.83 140.97 90)
 			(effects
@@
 			)
 		)
-		(property "Manufacturer" "Samsung Electro-Mechanics"
+		(property "Manufacturer" "Yageo"
 			(at 36.83 140.97 0)
 			(effects
@@
 			)
 		)
-		(property "MPN" "CL21B104KCFNNNE"
+		(property "MPN" "CC0805KKX7R0BB104"
 			(at 36.83 140.97 0)
 			(effects
@@
 			)
 		)
-		(property "Description" "C28233"
+		(property "Description" "C106243"
 			(at 66.04 168.91 0)
 			(effects
@@
 			)
 		)
-		(property "LCSC" "C28233"
+		(property "LCSC" "C106243"
 			(at 66.04 168.91 90)
 			(effects
@@
 			)
 		)
-		(property "Manufacturer" "Samsung Electro-Mechanics"
+		(property "Manufacturer" "Yageo"
 			(at 66.04 168.91 0)
 			(effects
@@
 			)
 		)
-		(property "MPN" "CL21B104KCFNNNE"
+		(property "MPN" "CC0805KKX7R0BB104"
 			(at 66.04 168.91 0)
 			(effects
@@
 			)
 		)
-		(property "Description" "C28233"
+		(property "Description" "C106243"
 			(at 363.22 53.34 0)
 			(effects
@@
 			)
 		)
-		(property "LCSC" "C28233"
+		(property "LCSC" "C106243"
 			(at 363.22 53.34 0)
 			(effects
@@
 			)
 		)
-		(property "Manufacturer" "Samsung Electro-Mechanics"
+		(property "Manufacturer" "Yageo"
 			(at 363.22 53.34 0)
 			(effects
@@
 			)
 		)
-		(property "MPN" "CL21B104KCFNNNE"
+		(property "MPN" "CC0805KKX7R0BB104"
 			(at 363.22 53.34 0)
 			(effects
@@
 			)
 		)
-		(property "Description" "C28233"
+		(property "Description" "C106243"
 			(at 64.77 36.83 0)
 			(effects
@@
 			)
 		)
-		(property "LCSC" "C28233"
+		(property "LCSC" "C106243"
 			(at 64.77 36.83 90)
 			(effects
@@
 			)
 		)
-		(property "Manufacturer" "Samsung Electro-Mechanics"
+		(property "Manufacturer" "Yageo"
 			(at 64.77 36.83 0)
 			(effects
@@
 			)
 		)
-		(property "MPN" "CL21B104KCFNNNE"
+		(property "MPN" "CC0805KKX7R0BB104"
 			(at 64.77 36.83 0)
 			(effects
@@
 			)
 		)
-		(property "Description" "C28233"
+		(property "Description" "C106243"
 			(at 314.96 53.34 0)
 			(effects
@@
 			)
 		)
-		(property "LCSC" "C28233"
+		(property "LCSC" "C106243"
 			(at 314.96 53.34 0)
 			(effects
@@
 			)
 		)
-		(property "Manufacturer" "Samsung Electro-Mechanics"
+		(property "Manufacturer" "Yageo"
 			(at 314.96 53.34 0)
 			(effects
@@
 			)
 		)
-		(property "MPN" "CL21B104KCFNNNE"
+		(property "MPN" "CC0805KKX7R0BB104"
 			(at 314.96 53.34 0)
 			(effects
@@
 			)
 		)
-		(property "Description" "C28233"
+		(property "Description" "C106243"
 			(at 87.63 36.83 0)
 			(effects
@@
 			)
 		)
-		(property "LCSC" "C28233"
+		(property "LCSC" "C106243"
 			(at 87.63 36.83 90)
 			(effects
@@
 			)
 		)
-		(property "Manufacturer" "Samsung Electro-Mechanics"
+		(property "Manufacturer" "Yageo"
 			(at 87.63 36.83 0)
 			(effects
@@
 			)
 		)
-		(property "MPN" "CL21B104KCFNNNE"
+		(property "MPN" "CC0805KKX7R0BB104"
 			(at 87.63 36.83 0)
 			(effects
@@
 			)
 		)
-		(property "Description" "Samsung CL21B105KBFNNNE 1 uF 50 V X7R 0805 MLCC"
+		(property "Description" "Yageo CC0805KKX7R9BB105 1 uF 50 V X7R 0805 MLCC"
 			(at 37.465 168.275 0)
 			(effects
@@
 			)
 		)
-		(property "LCSC" "C28323"
+		(property "LCSC" "C91185"
 			(at 37.465 168.275 90)
 			(effects
@@
 			)
 		)
-		(property "Manufacturer" "Samsung"
+		(property "Manufacturer" "Yageo"
 			(at 37.465 168.275 0)
 			(effects
@@
 			)
 		)
-		(property "MPN" "CL21B105KBFNNNE"
+		(property "MPN" "CC0805KKX7R9BB105"
 			(at 37.465 168.275 0)
 			(effects
@@
 			)
 		)
-		(property "Description" "C28233"
+		(property "Description" "C106243"
 			(at 41.91 36.83 0)
 			(effects
@@
 			)
 		)
-		(property "LCSC" "C28233"
+		(property "LCSC" "C106243"
 			(at 41.91 36.83 90)
 			(effects
@@
 			)
 		)
-		(property "Manufacturer" "Samsung Electro-Mechanics"
+		(property "Manufacturer" "Yageo"
 			(at 41.91 36.83 0)
 			(effects
@@
 			)
 		)
-		(property "MPN" "CL21B104KCFNNNE"
+		(property "MPN" "CC0805KKX7R0BB104"
 			(at 41.91 36.83 0)
 			(effects
@@
 			)
 		)
-		(property "Description" "C28233"
+		(property "Description" "C106243"
 			(at 50.8 167.64 0)
 			(effects
@@
 			)
 		)
-		(property "LCSC" "C28233"
+		(property "LCSC" "C106243"
 			(at 50.8 167.64 90)
 			(effects
@@
 			)
 		)
-		(property "Manufacturer" "Samsung Electro-Mechanics"
+		(property "Manufacturer" "Yageo"
 			(at 50.8 167.64 0)
 			(effects
@@
 			)
 		)
-		(property "MPN" "CL21B104KCFNNNE"
+		(property "MPN" "CC0805KKX7R0BB104"
 			(at 50.8 167.64 0)
 			(effects
@@
 			)
 		)
-		(property "Description" "Samsung CL21B105KBFNNNE 1 uF 50 V X7R 0805 MLCC; DC-bias derating requires prototype measurement and datasheet-curve verification before release"
+		(property "Description" "Yageo CC0805KKX7R9BB105 1 uF 50 V X7R 0805 MLCC; DC-bias derating requires prototype measurement and datasheet-curve verification before release"
 			(at 228.6 15.24 0)
 			(hide yes)
@@
 			)
 		)
-		(property "LCSC" "C28323"
+		(property "LCSC" "C91185"
 			(at 228.6 15.24 0)
 			(hide yes)
@@
 			)
 		)
-		(property "Manufacturer" "Samsung"
+		(property "Manufacturer" "Yageo"
 			(at 228.6 15.24 0)
 			(hide yes)
@@
 			)
 		)
-		(property "MPN" "CL21B105KBFNNNE"
+		(property "MPN" "CC0805KKX7R9BB105"
 			(at 228.6 15.24 0)
 			(hide yes)
@@
 			)
 		)
-		(property "Description" "Samsung CL21B105KBFNNNE 1 uF 50 V X7R 0805 MLCC; DC-bias derating requires prototype measurement and datasheet-curve verification before release"
+		(property "Description" "Yageo CC0805KKX7R9BB105 1 uF 50 V X7R 0805 MLCC; DC-bias derating requires prototype measurement and datasheet-curve verification before release"
 			(at 228.6 55.88 0)
 			(hide yes)
@@
 			)
 		)
-		(property "LCSC" "C28323"
+		(property "LCSC" "C91185"
 			(at 228.6 55.88 0)
 			(hide yes)
@@
 			)
 		)
-		(property "Manufacturer" "Samsung"
+		(property "Manufacturer" "Yageo"
 			(at 228.6 55.88 0)
 			(hide yes)
@@
 			)
 		)
-		(property "MPN" "CL21B105KBFNNNE"
+		(property "MPN" "CC0805KKX7R9BB105"
 			(at 228.6 55.88 0)
 			(hide yes)
@@
 			)
 		)
-		(property "Datasheet" "https://datasheet.lcsc.com/lcsc/1912111437_UNI-ROYAL-Uniroyal-Elec-0805W8F1002T5E_C17414.pdf"
+		(property "Datasheet" "https://jlcpcb.com/partdetail/UNIROYAL-0805W8F1002T5E/C17414"
 			(at 314.96 38.1 0)
 			(hide yes)
@@
 			)
 		)
-		(property "Description" "10 kOhm, 1%, 0805; JLCPCB C17414"
+		(property "Description" "UNI-ROYAL 0805W8F1002T5E 10 kOhm 1% 1/8 W 0805 thick-film resistor"
 			(at 314.96 38.1 0)
 			(hide yes)
@@
 			)
 		)
-		(property "Datasheet" "https://datasheet.lcsc.com/lcsc/1912111437_UNI-ROYAL-Uniroyal-Elec-0805W8F1002T5E_C17414.pdf"
+		(property "Datasheet" "https://jlcpcb.com/partdetail/UNIROYAL-0805W8F1002T5E/C17414"
 			(at 325.12 55.88 0)
 			(hide yes)
@@
 			)
 		)
-		(property "Description" "10 kOhm, 1%, 0805; JLCPCB C17414"
+		(property "Description" "UNI-ROYAL 0805W8F1002T5E 10 kOhm 1% 1/8 W 0805 thick-film resistor"
 			(at 325.12 55.88 0)
 			(hide yes)
@@
 			)
 		)
-		(property "Datasheet" "https://datasheet.lcsc.com/lcsc/1912111437_UNI-ROYAL-Uniroyal-Elec-0805W8F1002T5E_C17414.pdf"
+		(property "Datasheet" "https://jlcpcb.com/partdetail/UNIROYAL-0805W8F1002T5E/C17414"
 			(at 345.44 55.88 0)
 			(hide yes)
@@
 			)
 		)
-		(property "Description" "10 kOhm, 1%, 0805; JLCPCB C17414"
+		(property "Description" "UNI-ROYAL 0805W8F1002T5E 10 kOhm 1% 1/8 W 0805 thick-film resistor"
 			(at 345.44 55.88 0)
 			(hide yes)
@@
 			)
 		)
-		(property "Datasheet" "https://datasheet.lcsc.com/lcsc/1912111437_Samsung-Electro-Mechanics-CL21B104KCFNNNE_C28233.pdf"
+		(property "Datasheet" "https://jlcpcb.com/partdetail/Yageo-CC0805KKX7R0BB104/C106243"
 			(at 269.24 38.1 0)
 			(hide yes)
@@
 			)
 		)
-		(property "Description" "100 nF, 100 V, X7R, 0805; JLCPCB C28233"
+		(property "Description" "100 nF, 100 V, X7R, 10%, 0805; JLCPCB C106243"
 			(at 269.24 38.1 0)
 			(hide yes)
@@
 			)
 		)
-		(property "LCSC" "C28233"
+		(property "LCSC" "C106243"
 			(at 0 0 0)
 			(effects
@@
 			)
 		)
-		(property "Manufacturer" "Samsung Electro-Mechanics"
+		(property "Manufacturer" "Yageo"
 			(at 0 0 0)
 			(effects
@@
 			)
 		)
-		(property "MPN" "CL21B104KCFNNNE"
+		(property "MPN" "CC0805KKX7R0BB104"
 			(at 0 0 0)
 			(effects
@@
 			)
 		)
-		(property "Datasheet" "https://datasheet.lcsc.com/lcsc/1912111437_Samsung-Electro-Mechanics-CL21B104KCFNNNE_C28233.pdf"
+		(property "Datasheet" "https://jlcpcb.com/partdetail/Yageo-CC0805KKX7R0BB104/C106243"
 			(at 269.24 76.2 0)
 			(hide yes)
@@
 			)
 		)
-		(property "Description" "100 nF, 100 V, X7R, 0805; JLCPCB C28233"
+		(property "Description" "100 nF, 100 V, X7R, 10%, 0805; JLCPCB C106243"
 			(at 269.24 76.2 0)
 			(hide yes)
@@
 			)
 		)
-		(property "LCSC" "C28233"
+		(property "LCSC" "C106243"
 			(at 0 0 0)
 			(effects
@@
 			)
 		)
-		(property "Manufacturer" "Samsung Electro-Mechanics"
+		(property "Manufacturer" "Yageo"
 			(at 0 0 0)
 			(effects
@@
 			)
 		)
-		(property "MPN" "CL21B104KCFNNNE"
+		(property "MPN" "CC0805KKX7R0BB104"
 			(at 0 0 0)
 			(effects

Commit message: feat(pcb): finish rev3a connector integration
Parts:
- J2: value 1x6 -> RECOVERY; footprint Connector_PinHeader_2.54mm:PinHeader_1x06_P2.54mm_Vertical -> OnionStraws:Recovery_Header_2x3_P2.54mm_Vertical; LCSC (none) -> C42391552; MPN (none) -> HX PZ-2.54-02-03-S-PB3.2; Manufacturer (none) -> hanxia; now fitted; now in the parts list
Changed lines of the file:
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@@
 		(exclude_from_sim no)
 		(in_bom no)
-		(on_board yes)
+		(on_board no)
 		(dnp yes)
 		(fields_autoplaced yes)
@@
 			)
 		)
-		(property "Description" "DNP connector-free Tag-Connect recovery footprint; manual flash fallback when USB is unavailable; no installed part"
+		(property "Description" "DNP schematic alternate retained for reference; Rev3A uses populated J2 for recovery"
 			(at 49.53 232.41 0)
 			(effects
@@
 		(unit 1)
 		(exclude_from_sim no)
-		(in_bom no)
-		(on_board no)
-		(dnp yes)
+		(in_bom yes)
+		(on_board yes)
+		(dnp no)
 		(fields_autoplaced yes)
 		(property "Reference" "J2"
@@
 			)
 		)
-		(property "Value" "1x6"
+		(property "Value" "RECOVERY"
 			(at 52.07 214.6299 0)
 			(effects
@@
 			)
 		)
-		(property "Footprint" "Connector_PinHeader_2.54mm:PinHeader_1x06_P2.54mm_Vertical"
+		(property "Footprint" "OnionStraws:Recovery_Header_2x3_P2.54mm_Vertical"
 			(at 49.53 212.09 0)
 			(effects
@@
 			)
 		)
-		(property "Datasheet" "~"
+		(property "Datasheet" "https://jlcpcb.com/partdetail/hanxia-HX_PZ_2_54_02_03_S_PB32/C42391552"
 			(at 49.53 212.09 0)
 			(effects
@@
 			)
 		)
-		(property "Description" "Schematic-only diagnostic header; not placed on PCB (on_board no); do not install"
+		(property "Description" "Populated surface-mount 2x3, 2.54 mm male recovery header for 3.3 V UART flashing"
 			(at 49.53 212.09 0)
 			(effects
+				(font
+					(size 1.27 1.27)
+				)
+				(hide yes)
+			)
+		)
+		(property "MPN" "HX PZ-2.54-02-03-S-PB3.2"
+			(at 49.53 212.09 0)
+			(effects
+				(font
+					(size 1.27 1.27)
+				)
+				(hide yes)
+			)
+		)
+		(property "Manufacturer" "hanxia"
+			(at 49.53 212.09 0)
+			(effects
+				(font
+					(size 1.27 1.27)
+				)
+				(hide yes)
+			)
+		)
+		(property "LCSC" "C42391552"
+			(at 49.53 212.09 0)
+			(effects

Commit message: fix(pcb): complete rev3a review models
Other:
- company: (none) -> Dr-Crow
Changed lines of the file:
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@@
 		(date "2026-09-15")
 		(rev "3A")
+		(company "Dr-Crow")
+		(comment 1 "UNQUALIFIED PROTOTYPE - REVIEW BEFORE FABRICATION")
 	)
 	(junction
