File: pcb/OnionStraws.kicad_pcb (KiCad board)
At the start: 2 copper layers, 88.6 x 30 mm, 74 parts, among them J1 8P8C, J2 1x6, J3 TC2030, Q1 Si2309CDS, Q2 Si2309CDS, SW1 SW_Push, SW2 SW_Push, U1 APX803L20-29SA-7, U2 ESP32-C3-WROOM-02, U3 L7805, U4 74LVC2G07, U5 74LVC2G07_3v3, U6 AP2205-3.3

Commit message: fix(pcb): prepare revision 2.2 corrections
Parts:
- J1: footprint Connector_RJ:RJ45_Amphenol_54602-x08_Horizontal -> OnionStraws:RJ45_EVERCOM_5301-8P8C_Horizontal
Other:
- board text added: "5V 3v3 Half (7) Full TX (5) Full RX (4) GND"
- board text added: "mulcmu Onion Straws Revision 2.2"
- board text removed: "5V 3v3 Half (7) Full RX (5) Full TX (4) GND"
- board text removed: "mulcmu Onion Straws Revision 2.1"
Changed lines of the file:
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@@
 		(sheetname "/")
 		(sheetfile "OnionStraws.kicad_sch")
-		(attr smd)
+		(attr smd exclude_from_pos_files exclude_from_bom dnp)
 		(fp_line
 			(start 0 -1.56)
@@
 		)
 	)
-	(footprint "Connector_RJ:RJ45_Amphenol_54602-x08_Horizontal"
+	(footprint "OnionStraws:RJ45_EVERCOM_5301-8P8C_Horizontal"
 		(layer "F.Cu")
 		(at 122.425 99.2825 90)
-		(descr "8 Pol Shallow Latch Connector, Modjack, RJ45 (https://cdn.amphenol-icc.com/media/wysiwyg/files/drawing/c-bmj-0102.pdf)")
-		(tags "RJ45")
+		(descr "EVERCOM 5301-8P8C horizontal through-hole 8P8C jack, LCSC C3097717. Signal drills are 0.90 mm per the connector requirement.")
+		(tags "RJ45 8P8C EVERCOM 5301-8P8C")
 		(property "Reference" "J1"
 			(at 4.445 -5 90)
@@
 			(at 0 0 90)
 			(size 1.5 1.5)
-			(drill 0.76)
+			(drill 0.9)
 			(layers "*.Cu" "*.Mask")
 			(remove_unused_layers no)
@@
 			(at 1.27 -2.54 90)
 			(size 1.5 1.5)
-			(drill 0.76)
+			(drill 0.9)
 			(layers "*.Cu" "*.Mask")
 			(remove_unused_layers no)
@@
 			(at 2.54 0 90)
 			(size 1.5 1.5)
-			(drill 0.76)
+			(drill 0.9)
 			(layers "*.Cu" "*.Mask")
 			(remove_unused_layers no)
@@
 			(at 3.81 -2.54 90)
 			(size 1.5 1.5)
-			(drill 0.76)
+			(drill 0.9)
 			(layers "*.Cu" "*.Mask")
 			(remove_unused_layers no)
@@
 			(at 5.08 0 90)
 			(size 1.5 1.5)
-			(drill 0.76)
+			(drill 0.9)
 			(layers "*.Cu" "*.Mask")
 			(remove_unused_layers no)
@@
 			(at 6.35 -2.54 90)
 			(size 1.5 1.5)
-			(drill 0.76)
+			(drill 0.9)
 			(layers "*.Cu" "*.Mask")
 			(remove_unused_layers no)
@@
 			(at 7.62 0 90)
 			(size 1.5 1.5)
-			(drill 0.76)
+			(drill 0.9)
 			(layers "*.Cu" "*.Mask")
 			(remove_unused_layers no)
@@
 			(at 8.89 -2.54 90)
 			(size 1.5 1.5)
-			(drill 0.76)
+			(drill 0.9)
 			(layers "*.Cu" "*.Mask")
 			(remove_unused_layers no)
@@
 		)
 	)
-	(gr_text "mulcmu\nOnion Straws\nRevision 2.1"
+	(gr_text "mulcmu\nOnion Straws\nRevision 2.2"
 		(at 77.6 89.193091 0)
 		(layer "B.SilkS")
@@
 		)
 	)
-	(gr_text "5V\n\n\n3v3\n\n\nHalf (7)\n\n\nFull RX (5)\n\n\nFull TX (4)\n\n\nGND"
+	(gr_text "5V\n\n\n3v3\n\n\nHalf (7)\n\n\nFull TX (5)\n\n\nFull RX (4)\n\n\nGND"
 		(at 118.4 86 90)
 		(layer "B.SilkS")
