File: pcb/OnionStraws.kicad_sch (KiCad schematic)
At the start: 74 parts, among them J1 8P8C, J2 1x6, J3 TC2030, Q1 Si2309CDS, Q2 Si2309CDS, SW1 SW_Push, SW2 SW_Push, U1 APX803L20-29SA-7, U2 ESP32-C3-WROOM-02, U3 L7805, U4 74LVC2G07, U5 74LVC2G07_3v3, U6 AP2205-3.3

Commit message: fix(pcb): prepare revision 2.2 corrections
Parts:
- J1: footprint Connector_RJ:RJ45_Amphenol_54602-x08_Horizontal -> OnionStraws:RJ45_EVERCOM_5301-8P8C_Horizontal
- Q1: LCSC (none) -> C10493
- U1: now not fitted; now left out of the parts list
Changed lines of the file:
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@@
 			)
 		)
-		(property "Footprint" "Connector_RJ:RJ45_Amphenol_54602-x08_Horizontal"
+		(property "Footprint" "OnionStraws:RJ45_EVERCOM_5301-8P8C_Horizontal"
 			(at 43.815 94.615 90)
 			(effects
@@
 		(unit 1)
 		(exclude_from_sim no)
-		(in_bom yes)
+		(in_bom no)
 		(on_board yes)
-		(dnp no)
+		(dnp yes)
 		(fields_autoplaced yes)
 		(property "Reference" "U1"
@@
 			)
 		)
-		(property "LCSC" ""
+		(property "LCSC" "C10493"
 			(at 196.215 45.72 90)
 			(effects

Commit message: docs(pcb): polish revision 2.2 review package
Other:
- note added: "2.2 changes DNP U1 voltage supervisor Correct J1 RX/TX labels EVERCOM J1 footprint 0.90 mm signal drills"
- note removed: "2.1 changes Added ground test point Change D8 to bigger part move rj45 inboard 4.5mm smaller 7805 or different ldo"
Changed lines of the file:
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@@
 	(title_block
 		(title "Onion Straws")
-		(date "2025-05-22")
-		(rev "2.0")
+		(date "2026-09-14")
+		(rev "2.2")
 	)
 	(text "Voltage Supervisor, Hold ESP reset\nfor 150ms after power reaches 2.9V.\nPrevent brownout at boot."
@@
 		)
 	)
-	(text "2.1 changes\n\nAdded ground test point\nChange D8 to bigger part\n\nmove  rj45 inboard 4.5mm\nsmaller 7805 or different ldo"
+	(text "2.2 changes\n\nDNP U1 voltage supervisor\nCorrect J1 RX/TX labels\n\nEVERCOM J1 footprint\n0.90 mm signal drills"
 		(exclude_from_sim no)
 		(at 402.844 248.412 0)

Commit message: docs(pcb): finalize revision 2.2 orderability data
Parts:
- R18, R21: LCSC C17539 -> C104108
- R22: LCSC C17713 -> C17673
Changed lines of the file:
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@@
 			)
 		)
-		(property "Description" "C17713"
+		(property "Description" "C17673"
 			(at 344.805 133.35 0)
 			(effects
@@
 			)
 		)
-		(property "LCSC" "C17713"
+		(property "LCSC" "C17673"
 			(at 344.805 133.35 90)
 			(effects
@@
 			)
 		)
-		(property "Description" "C17539"
+		(property "Description" "C104108"
 			(at 335.915 179.705 0)
 			(effects
@@
 			)
 		)
-		(property "LCSC" "C17539"
+		(property "LCSC" "C104108"
 			(at 335.915 179.705 90)
 			(effects
@@
 			)
 		)
-		(property "Description" "C17539"
+		(property "Description" "C104108"
 			(at 335.915 118.745 0)
 			(effects
@@
 			)
 		)
-		(property "LCSC" "C17539"
+		(property "LCSC" "C104108"
 			(at 335.915 118.745 90)
 			(effects
