File: pcb/rev3b/design/GEA-Adapter-Rev3B.kicad_pcb (KiCad board)
At the start: 4 copper layers, 99 x 40 mm, 99 parts, among them J1 8P8C, J2 RECOVERY, Q3 CJ3407, Q4 CJ3407, Q5 MMBT3904, U10 TPS22810DBVR, U2 XIAO ESP32-C3 v1.3 (22-pad), U4 74LVC2G07, U5 74LVC2G07_3v3, U8 AP63205WU, U9 TPS22810DBVR

Commit message: fix(pcb): connect Rev3B LED and recovery signals
Routing:
- net /LED2: track 0.00 -> 125.5 mm, vias 0 -> 2
- net EN: track 24.0 -> 120.9 mm, vias 2 -> 3
- net BOOT: track 67.5 -> 129.6 mm, vias 4 -> 5
Changed lines of the file:
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@@
 	)
 	(segment
+		(start 13.0257 26.7831)
+		(end 13.0257 27.1248)
+		(width 0.2)
+		(layer "F.Cu")
+		(net 6)
+	)
+	(segment
+		(start 92.97 4.835)
+		(end 91.5208 3.3858)
+		(width 0.2)
+		(layer "F.Cu")
+		(net 6)
+	)
+	(segment
+		(start 15.1826 24.6262)
+		(end 13.0257 26.7831)
+		(width 0.2)
+		(layer "F.Cu")
+		(net 6)
+	)
+	(segment
+		(start 91.5208 3.3858)
+		(end 91.5208 2.5196)
+		(width 0.2)
+		(layer "F.Cu")
+		(net 6)
+	)
+	(via
+		(at 91.5208 2.5196)
+		(size 0.8)
+		(drill 0.4)
+		(layers "F.Cu" "B.Cu")
+		(net 6)
+	)
+	(via
+		(at 15.1826 24.6262)
+		(size 0.8)
+		(drill 0.4)
+		(layers "F.Cu" "B.Cu")
+		(net 6)
+	)
+	(segment
+		(start 15.6806 38.9276)
+		(end 10.6195 33.8665)
+		(width 0.2)
+		(layer "In2.Cu")
+		(net 6)
+	)
+	(segment
+		(start 91.5208 2.5196)
+		(end 91.5208 18.9785)
+		(width 0.2)
+		(layer "In2.Cu")
+		(net 6)
+	)
+	(segment
+		(start 91.5208 18.9785)
+		(end 71.5717 38.9276)
+		(width 0.2)
+		(layer "In2.Cu")
+		(net 6)
+	)
+	(segment
+		(start 14.5339 24.6262)
+		(end 15.1826 24.6262)
+		(width 0.2)
+		(layer "In2.Cu")
+		(net 6)
+	)
+	(segment
+		(start 71.5717 38.9276)
+		(end 15.6806 38.9276)
+		(width 0.2)
+		(layer "In2.Cu")
+		(net 6)
+	)
+	(segment
+		(start 10.6195 33.8665)
+		(end 10.6195 28.5406)
+		(width 0.2)
+		(layer "In2.Cu")
+		(net 6)
+	)
+	(segment
+		(start 10.6195 28.5406)
+		(end 14.5339 24.6262)
+		(width 0.2)
+		(layer "In2.Cu")
+		(net 6)
+	)
+	(segment
 		(start 87.89 23.1312)
 		(end 87.89 21)
@@
 	)
 	(segment
+		(start 14.43 29.96)
+		(end 12.3483 29.96)
+		(width 0.2)
+		(layer "F.Cu")
+		(net 51)
+	)
+	(segment
+		(start 12.3483 29.712)
+		(end 11.3999 28.7636)
+		(width 0.2)
+		(layer "F.Cu")
+		(net 51)
+	)
+	(segment
 		(start 59.6885 37.8885)
 		(end 58.8 37)
@@
 	)
 	(segment
+		(start 12.3483 29.96)
+		(end 12.3483 29.712)
+		(width 0.2)
+		(layer "F.Cu")
+		(net 51)
+	)
+	(segment
 		(start 65.0729 35.2095)
 		(end 62.3939 37.8885)
@@
 	)
 	(via
+		(at 11.3999 28.7636)
+		(size 0.8)
+		(drill 0.4)
+		(layers "F.Cu" "B.Cu")
+		(net 51)
+	)
+	(via
 		(at 65.0729 35.2095)
 		(size 0.8)
@@
 	)
 	(segment
+		(start 65.0729 35.2095)
+		(end 14.2253 35.2095)
+		(width 0.2)
+		(layer "In2.Cu")
+		(net 51)
+	)
+	(segment
 		(start 26.3714 11.6514)
 		(end 27.7653 10.2575)
@@
 	)
 	(segment
+		(start 14.2253 35.2095)
+		(end 11.3999 32.3841)
+		(width 0.2)
+		(layer "In2.Cu")
+		(net 51)
+	)
+	(segment
 		(start 26.3714 18.5764)
 		(end 26.3714 11.6514)
@@
 	)
 	(segment
+		(start 11.3999 32.3841)
+		(end 11.3999 28.7636)
+		(width 0.2)
+		(layer "In2.Cu")
+		(net 51)
+	)
+	(segment
 		(start 20.8795 24.0683)
 		(end 26.3714 18.5764)
@@
 	)
 	(segment
+		(start 8.97 35.04)
+		(end 11.0517 35.04)
+		(width 0.2)
+		(layer "F.Cu")
+		(net 53)
+	)
+	(segment
 		(start 92.6484 10.2864)
 		(end 87.1377 10.2864)
@@
 	)
 	(segment
+		(start 11.327 33.5479)
+		(end 11.327 34.7647)
+		(width 0.2)
+		(layer "F.Cu")
+		(net 53)
+	)
+	(segment
+		(start 11.327 34.7647)
+		(end 11.0517 35.04)
+		(width 0.2)
+		(layer "F.Cu")
+		(net 53)
+	)
+	(segment
 		(start 87.1377 10.2864)
 		(end 84.4402 7.5889)
@@
 		(net 53)
 	)
+	(via
+		(at 11.327 33.5479)
+		(size 0.8)
+		(drill 0.4)
+		(layers "F.Cu" "B.Cu")
+		(net 53)
+	)
+	(segment
+		(start 82.8477 19.6246)
+		(end 64.1847 38.2876)
+		(width 0.2)
+		(layer "In2.Cu")
+		(net 53)
+	)
 	(segment
 		(start 81.4072 2.8317)
@@
 	)
 	(segment
+		(start 64.1847 38.2876)
+		(end 16.0667 38.2876)
+		(width 0.2)
+		(layer "In2.Cu")
+		(net 53)
+	)
+	(segment
+		(start 82.8477 7.5889)
+		(end 82.8477 19.6246)
+		(width 0.2)
+		(layer "In2.Cu")
+		(net 53)
+	)
+	(segment
 		(start 82.8477 4.2722)
 		(end 82.8477 7.5889)
 		(width 0.2)
 		(layer "In2.Cu")
+		(net 53)
+	)
+	(segment
+		(start 16.0667 38.2876)
+		(end 11.327 33.5479)
+		(width 0.2)
+		(layer "In2.Cu")

Commit message: fix(pcb): connect Rev3B capacitor ground island
Routing:
- net GND: vias 8 -> 9
Changed lines of the file:
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@@
+		(net 14)
+	)
+	(via
+		(at 16.7 24.65)
+		(size 0.8)
+		(drill 0.4)
+		(layers "F.Cu" "B.Cu")
 		(net 14)
 	)

Commit message: fix(pcb): connect Rev3B decoupling capacitor ground
Routing:
- net GND: vias 9 -> 10
Changed lines of the file:
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@@
+		(net 14)
+	)
+	(via
+		(at 23.6 29.2)
+		(size 0.8)
+		(drill 0.4)
+		(layers "F.Cu" "B.Cu")
 		(net 14)
 	)
