File: pcb/rev3b/design/GEA-Adapter-Rev3B.kicad_sch (KiCad schematic)
At the start: 103 parts, among them J1 8P8C, J2 RECOVERY, J3 TC2030, Q3 CJ3407, Q4 CJ3407, Q5 MMBT3904, U10 TPS1H200AQDGNRQ1, U2 XIAO ESP32-C3 v1.3 (22-pad), U4 74LVC2G07, U5 74LVC2G07_3v3, U8 AP63205WU, U9 TPS1H200AQDGNRQ1

Commit message: fix(pcb): record complete Murata capacitor ordering identities
Parts:
- C15: MPN GCM188L81H104KA57 -> GCM188L81H104KA57D
Changed lines of the file:
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@@
 			)
 		)
-		(property "MPN" "GCM188L81H104KA57"
+		(property "MPN" "GCM188L81H104KA57D"
 			(at 269.24 91.44 0)
 			(effects

Commit message: fix(pcb): backport Rev3B input diode rating repair
Parts:
- D14, D15: value MBR0540-TP -> STPS140Z; LCSC C78744 -> C155662; MPN MBR0540-TP -> STPS140Z; Manufacturer MCC -> STMicroelectronics
Changed lines of the file:
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@@
 			)
 		)
-		(property "Value" "MBR0540-TP"
+		(property "Value" "STPS140Z"
 			(at 299.72 35.56 0)
 			(show_name no)
@@
 			)
 		)
-		(property "Datasheet" "https://www.mccsemi.com/up_pdf/MBR0520~MBR0580(SOD123).pdf"
+		(property "Datasheet" "https://www.st.com/resource/en/datasheet/stps140z.pdf"
 			(at 284.48 25.4 0)
 			(hide yes)
@@
 			)
 		)
-		(property "Description" "40 V, 0.5 A Schottky rectifier, SOD-123; JLCPCB C78744"
+		(property "Description" "40 V, 1 A Schottky rectifier, SOD-123; maximum junction 150 degC; LCSC C155662"
 			(at 284.48 25.4 0)
 			(hide yes)
@@
 			)
 		)
-		(property "LCSC" "C78744"
+		(property "LCSC" "C155662"
 			(at 0 0 0)
 			(effects
@@
 			)
 		)
-		(property "Manufacturer" "MCC"
+		(property "Manufacturer" "STMicroelectronics"
 			(at 0 0 0)
 			(effects
@@
 			)
 		)
-		(property "MPN" "MBR0540-TP"
+		(property "MPN" "STPS140Z"
 			(at 0 0 0)
 			(effects
@@
 			)
 		)
-		(property "Value" "MBR0540-TP"
+		(property "Value" "STPS140Z"
 			(at 299.72 96.52 0)
 			(show_name no)
@@
 			)
 		)
-		(property "Datasheet" "http://www.mccsemi.com/up_pdf/MBR0520~MBR0580(SOD123).pdf"
+		(property "Datasheet" "https://www.st.com/resource/en/datasheet/stps140z.pdf"
 			(at 284.48 63.5 0)
 			(hide yes)
@@
 			)
 		)
-		(property "Description" "40V 0.5A Schottky Power Rectifier Diode, SOD-123"
+		(property "Description" "40 V, 1 A Schottky rectifier, SOD-123; maximum junction 150 degC; LCSC C155662"
 			(at 284.48 63.5 0)
 			(hide yes)
@@
 			)
 		)
-		(property "LCSC" "C78744"
+		(property "LCSC" "C155662"
 			(at 0 0 0)
 			(effects
@@
 			)
 		)
-		(property "Manufacturer" "MCC"
+		(property "Manufacturer" "STMicroelectronics"
 			(at 0 0 0)
 			(effects
@@
 			)
 		)
-		(property "MPN" "MBR0540-TP"
+		(property "MPN" "STPS140Z"
 			(at 0 0 0)
 			(effects
