File: pcb/rev1.0/design/OnionStraws.kicad_sch (KiCad schematic)
At the start: 61 parts, among them J1 Conn_01x04, J2 8P8C, Q1 Si2309CDS, Q2 Si2309CDS, SW1 SW_Push, U1 74LVC2G07, U2 74LVC2G07_3v3, U3 ESP32, U4 APX803L

Commit message: fix(pcb): correct legacy assembly and regulator metadata
Parts:
- H1, H2, H3, H4, TP1, TP2, TP3, TP4, TP5, TP6, TP7: now left out of the parts list
- R1: now not fitted; now left out of the parts list
Changed lines of the file:
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@@
   )
   (symbol (lib_id "LegacySymbols:MountingHole") (at 223.52 228.6 0) (unit 1)
-    (in_bom yes) (on_board yes) (fields_autoplaced)
+    (in_bom no) (on_board yes) (fields_autoplaced)
     (property "Reference" "H3" (id 0) (at 226.06 227.6915 0)
       (effects (font (size 1.27 1.27)) (justify left))
@@
   )
   (symbol (lib_id "LegacySymbols:TestPoint") (at 135.255 100.33 0) (unit 1)
-    (in_bom yes) (on_board yes) (fields_autoplaced)
+    (in_bom no) (on_board yes) (fields_autoplaced)
     (property "Reference" "TP3" (id 0) (at 136.652 96.1195 0)
       (effects (font (size 1.27 1.27)) (justify left))
@@
   )
   (symbol (lib_id "LegacySymbols:TestPoint") (at 37.465 139.065 0) (unit 1)
-    (in_bom yes) (on_board yes) (fields_autoplaced)
+    (in_bom no) (on_board yes) (fields_autoplaced)
     (property "Reference" "TP5" (id 0) (at 38.862 134.8545 0)
       (effects (font (size 1.27 1.27)) (justify left))
@@
   )
   (symbol (lib_id "LegacySymbols:MountingHole") (at 200.025 221.615 0) (unit 1)
-    (in_bom yes) (on_board yes) (fields_autoplaced)
+    (in_bom no) (on_board yes) (fields_autoplaced)
     (property "Reference" "H1" (id 0) (at 202.565 220.7065 0)
       (effects (font (size 1.27 1.27)) (justify left))
@@
   )
   (symbol (lib_id "LegacySymbols:TestPoint") (at 125.095 26.035 0) (unit 1)
-    (in_bom yes) (on_board yes) (fields_autoplaced)
+    (in_bom no) (on_board yes) (fields_autoplaced)
     (property "Reference" "TP1" (id 0) (at 126.492 21.8245 0)
       (effects (font (size 1.27 1.27)) (justify left))
@@
   )
   (symbol (lib_id "LegacySymbols:TestPoint") (at 38.1 166.37 0) (unit 1)
-    (in_bom yes) (on_board yes) (fields_autoplaced)
+    (in_bom no) (on_board yes) (fields_autoplaced)
     (property "Reference" "TP7" (id 0) (at 39.497 162.1595 0)
       (effects (font (size 1.27 1.27)) (justify left))
@@
   )
   (symbol (lib_id "LegacySymbols:MountingHole") (at 224.155 221.615 0) (unit 1)
-    (in_bom yes) (on_board yes) (fields_autoplaced)
+    (in_bom no) (on_board yes) (fields_autoplaced)
     (property "Reference" "H2" (id 0) (at 226.695 220.7065 0)
       (effects (font (size 1.27 1.27)) (justify left))
@@
   )
   (symbol (lib_id "LegacySymbols:MountingHole") (at 200.025 229.235 0) (unit 1)
-    (in_bom yes) (on_board yes) (fields_autoplaced)
+    (in_bom no) (on_board yes) (fields_autoplaced)
     (property "Reference" "H4" (id 0) (at 202.565 228.3265 0)
       (effects (font (size 1.27 1.27)) (justify left))
@@
   )
   (symbol (lib_id "LegacySymbols:TestPoint") (at 235.585 123.825 0) (unit 1)
-    (in_bom yes) (on_board yes) (fields_autoplaced)
+    (in_bom no) (on_board yes) (fields_autoplaced)
     (property "Reference" "TP4" (id 0) (at 236.982 119.6145 0)
       (effects (font (size 1.27 1.27)) (justify left))
@@
   )
   (symbol (lib_id "LegacySymbols:TestPoint") (at 235.585 80.01 0) (unit 1)
-    (in_bom yes) (on_board yes) (fields_autoplaced)
+    (in_bom no) (on_board yes) (fields_autoplaced)
     (property "Reference" "TP2" (id 0) (at 236.982 75.7995 0)
       (effects (font (size 1.27 1.27)) (justify left))
@@
   )
   (symbol (lib_id "LegacySymbols:TestPoint") (at 236.855 140.97 0) (unit 1)
-    (in_bom yes) (on_board yes) (fields_autoplaced)
+    (in_bom no) (on_board yes) (fields_autoplaced)
     (property "Reference" "TP6" (id 0) (at 238.252 136.7595 0)
       (effects (font (size 1.27 1.27)) (justify left))
@@
   )
   (symbol (lib_id "LegacySymbols:R") (at 173.355 40.64 180) (unit 1)
-    (in_bom yes) (on_board yes)
+    (in_bom no) (on_board yes)
+		(dnp yes)
     (property "Reference" "R1" (id 0) (at 175.895 40.64 90))
     (property "Value" "DNP" (id 1) (at 173.355 40.64 90))
