File: pcb/rev2.0/design/OnionStraws.kicad_sch (KiCad schematic)
At the start: 75 parts, among them J1 8P8C, J2 1x6, J3 TC2030, Q1 Si2309CDS, Q2 Si2309CDS, SW1 SW_Push, SW2 SW_Push, U1 APX803L20-29SA-7, U2 ESP32-C3-WROOM-02, U3 L7805, U4 74LVC2G07, U5 74LVC2G07_3v3, U6 AP2205-3.3

Commit message: fix(pcb): correct legacy assembly and regulator metadata
Parts:
- H1, H2: now left out of the parts list
Changed lines of the file:
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@@
 		(unit 1)
 		(exclude_from_sim no)
-		(in_bom yes)
+		(in_bom no)
 		(on_board yes)
 		(dnp no)
@@
 			)
 		)
-		(property "Datasheet" "https://www.diodes.com/assets/Datasheets/products_inactive_data/AP2204.pdf"
+		(property "Datasheet" "https://www.diodes.com/assets/Datasheets/AP2205.pdf"
 			(at 337.82 43.18 0)
 			(effects
@@
 		(unit 1)
 		(exclude_from_sim no)
-		(in_bom yes)
+		(in_bom no)
 		(on_board yes)
 		(dnp no)
