File: pcb/rev2.2/design/OnionStraws.kicad_sch (KiCad schematic)
At the start: 74 parts, among them J1 8P8C, J2 1x6, J3 TC2030, Q1 Si2309CDS, Q2 Si2309CDS, SW1 SW_Push, SW2 SW_Push, U1 APX803L20-29SA-7, U2 ESP32-C3-WROOM-02, U3 L7805, U4 74LVC2G07, U5 74LVC2G07_3v3, U6 AP2205-3.3

Commit message: fix(pcb): stage reviewed historical Rev2.2 source
Parts:
- C1: footprint Capacitor_SMD:C_0805_2012Metric -> LegacyBoard:C1_C_0805_2012Metric; symbol Device:C -> LegacySymbols:C
- C10: footprint Capacitor_SMD:C_0805_2012Metric -> LegacyBoard:C10_C_0805_2012Metric; symbol Device:C -> LegacySymbols:C
- C11: footprint Capacitor_SMD:C_0805_2012Metric -> LegacyBoard:C11_C_0805_2012Metric; symbol Device:C -> LegacySymbols:C
- C12: footprint Capacitor_SMD:C_0805_2012Metric -> LegacyBoard:C12_C_0805_2012Metric; symbol Device:C -> LegacySymbols:C
- C13: footprint Capacitor_SMD:C_0805_2012Metric -> LegacyBoard:C13_C_0805_2012Metric; symbol Device:C -> LegacySymbols:C
- C14: footprint Capacitor_SMD:C_0805_2012Metric -> LegacyBoard:C14_C_0805_2012Metric; symbol Device:C -> LegacySymbols:C
- C2: footprint Capacitor_SMD:C_0805_2012Metric -> LegacyBoard:C2_C_0805_2012Metric; symbol Device:C -> LegacySymbols:C
- C3: footprint Capacitor_SMD:C_0805_2012Metric -> LegacyBoard:C3_C_0805_2012Metric; symbol Device:C -> LegacySymbols:C
- C4: footprint Capacitor_SMD:C_0805_2012Metric -> LegacyBoard:C4_C_0805_2012Metric; symbol Device:C -> LegacySymbols:C
- C5: footprint Capacitor_SMD:C_0805_2012Metric -> LegacyBoard:C5_C_0805_2012Metric; symbol Device:C -> LegacySymbols:C
- C6: footprint Capacitor_SMD:C_0805_2012Metric -> LegacyBoard:C6_C_0805_2012Metric; symbol Device:C -> LegacySymbols:C
- C7: footprint Capacitor_SMD:C_0805_2012Metric -> LegacyBoard:C7_C_0805_2012Metric; symbol Device:C -> LegacySymbols:C
- C8: footprint Capacitor_SMD:C_0805_2012Metric -> LegacyBoard:C8_C_0805_2012Metric; symbol Device:C -> LegacySymbols:C
- C9: footprint Capacitor_SMD:C_0805_2012Metric -> LegacyBoard:C9_C_0805_2012Metric; symbol Device:C -> LegacySymbols:C
- D1: footprint Package_TO_SOT_SMD:SOT-23 -> LegacyBoard:D1_SOT-23; symbol Diode:BAV99 -> LegacySymbols:BAV99
- D2: footprint Package_TO_SOT_SMD:SOT-23 -> LegacyBoard:D2_SOT-23; symbol Diode:BAV99 -> LegacySymbols:BAV99
- D3: footprint Package_TO_SOT_SMD:SOT-23 -> LegacyBoard:D3_SOT-23; symbol Diode:BAV99 -> LegacySymbols:BAV99
- D4: footprint LED_SMD:LED_0805_2012Metric -> LegacyBoard:D4_LED_0805_2012Metric; symbol Device:LED -> LegacySymbols:LED
- D5: footprint LED_SMD:LED_0805_2012Metric -> LegacyBoard:D5_LED_0805_2012Metric; symbol Device:LED -> LegacySymbols:LED
- D6: footprint LED_SMD:LED_0805_2012Metric -> LegacyBoard:D6_LED_0805_2012Metric; symbol Device:LED -> LegacySymbols:LED
- D7: footprint Diode_SMD:D_SMA -> LegacyBoard:D7_D_SMA; symbol Device:D_TVS -> LegacySymbols:D_TVS
- D8: footprint Diode_SMD:D_SOD-123 -> LegacyBoard:D8_D_SOD-123; symbol Device:D_Zener -> LegacySymbols:D_Zener
- D9: footprint Package_TO_SOT_SMD:SOT-23 -> LegacyBoard:D9_SOT-23; symbol Diode:BAV99 -> LegacySymbols:BAV99
- F1: footprint Fuse:Fuse_1812_4532Metric -> LegacyBoard:F1_Fuse_1812_4532Metric; symbol Device:Polyfuse -> LegacySymbols:Polyfuse
- F2: footprint Fuse:Fuse_1812_4532Metric -> LegacyBoard:F2_Fuse_1812_4532Metric; symbol Device:Polyfuse -> LegacySymbols:Polyfuse
- H1: footprint MountingHole:MountingHole_3.2mm_M3_DIN965 -> LegacyBoard:H1_MountingHole_3.2mm_M3_DIN965; symbol Mechanical:MountingHole -> LegacySymbols:MountingHole
- H2: footprint MountingHole:MountingHole_3.2mm_M3_DIN965 -> LegacyBoard:H2_MountingHole_3.2mm_M3_DIN965; symbol Mechanical:MountingHole -> LegacySymbols:MountingHole
- J1: footprint OnionStraws:RJ45_EVERCOM_5301-8P8C_Horizontal -> LegacyBoard:J1_RJ45_EVERCOM_5301-8P8C_Horizontal; symbol Connector:8P8C -> LegacySymbols:8P8C
- J2: footprint Connector_PinHeader_2.54mm:PinHeader_1x06_P2.54mm_Vertical -> LegacyBoard:J2_PinHeader_1x06_P2.54mm_Vertical; symbol Connector_Generic:Conn_01x06 -> LegacySymbols:Conn_01x06
- J3: footprint Connector:Tag-Connect_TC2030-IDC-NL_2x03_P1.27mm_Vertical -> LegacyBoard:J3_Tag-Connect_TC2030-IDC-NL_2x03_P1.27mm_Vertical; symbol Connector_Generic:Conn_01x06 -> LegacySymbols:Conn_01x06
- JP1: footprint Jumper:SolderJumper-3_P1.3mm_Bridged12_RoundedPad1.0x1.5mm_NumberLabels -> LegacyBoard:JP1_SolderJumper-3_P1.3mm_Bridged12_RoundedPad1.0x1.5mm_NumberLabels; symbol Jumper:SolderJumper_3_Bridged12 -> LegacySymbols:SolderJumper_3_Bridged12
- JP2: footprint Jumper:SolderJumper-3_P1.3mm_Bridged12_RoundedPad1.0x1.5mm_NumberLabels -> LegacyBoard:JP2_SolderJumper-3_P1.3mm_Bridged12_RoundedPad1.0x1.5mm_NumberLabels; symbol Jumper:SolderJumper_3_Bridged12 -> LegacySymbols:SolderJumper_3_Bridged12
- Q1: footprint Package_TO_SOT_SMD:SOT-23 -> LegacyBoard:Q1_SOT-23; symbol Device:Q_PMOS_GSD -> LegacySymbols:Q_PMOS_GSD
- Q2: footprint Package_TO_SOT_SMD:SOT-23 -> LegacyBoard:Q2_SOT-23; symbol Device:Q_PMOS_GSD -> LegacySymbols:Q_PMOS_GSD
- R1: footprint Resistor_SMD:R_0805_2012Metric -> LegacyBoard:R1_R_0805_2012Metric; symbol Device:R -> LegacySymbols:R
- R10: footprint Resistor_SMD:R_0805_2012Metric -> LegacyBoard:R10_R_0805_2012Metric; symbol Device:R -> LegacySymbols:R
- R11: footprint Resistor_SMD:R_0805_2012Metric -> LegacyBoard:R11_R_0805_2012Metric; symbol Device:R -> LegacySymbols:R
- R12: footprint Resistor_SMD:R_0805_2012Metric -> LegacyBoard:R12_R_0805_2012Metric; symbol Device:R -> LegacySymbols:R
- R13: footprint Resistor_SMD:R_0805_2012Metric -> LegacyBoard:R13_R_0805_2012Metric; symbol Device:R -> LegacySymbols:R
- R14: footprint Resistor_SMD:R_0805_2012Metric -> LegacyBoard:R14_R_0805_2012Metric; symbol Device:R -> LegacySymbols:R
- R15: footprint Resistor_SMD:R_0805_2012Metric -> LegacyBoard:R15_R_0805_2012Metric; symbol Device:R -> LegacySymbols:R
- R16: footprint Resistor_SMD:R_0805_2012Metric -> LegacyBoard:R16_R_0805_2012Metric; symbol Device:R -> LegacySymbols:R
- R17: footprint Resistor_SMD:R_0805_2012Metric -> LegacyBoard:R17_R_0805_2012Metric; symbol Device:R -> LegacySymbols:R
- R18: footprint Resistor_SMD:R_0805_2012Metric -> LegacyBoard:R18_R_0805_2012Metric; symbol Device:R -> LegacySymbols:R
- R19: footprint Resistor_SMD:R_0805_2012Metric -> LegacyBoard:R19_R_0805_2012Metric; symbol Device:R -> LegacySymbols:R
- R2: footprint Resistor_SMD:R_0805_2012Metric -> LegacyBoard:R2_R_0805_2012Metric; symbol Device:R -> LegacySymbols:R
- R20: footprint Resistor_SMD:R_0805_2012Metric -> LegacyBoard:R20_R_0805_2012Metric; symbol Device:R -> LegacySymbols:R
- R21: footprint Resistor_SMD:R_0805_2012Metric -> LegacyBoard:R21_R_0805_2012Metric; symbol Device:R -> LegacySymbols:R
- R22: footprint Resistor_SMD:R_0805_2012Metric -> LegacyBoard:R22_R_0805_2012Metric; symbol Device:R -> LegacySymbols:R
- R23: footprint Resistor_SMD:R_0805_2012Metric -> LegacyBoard:R23_R_0805_2012Metric; symbol Device:R -> LegacySymbols:R
- R24: footprint Resistor_SMD:R_0805_2012Metric -> LegacyBoard:R24_R_0805_2012Metric; symbol Device:R -> LegacySymbols:R
- R25: footprint Resistor_SMD:R_0805_2012Metric -> LegacyBoard:R25_R_0805_2012Metric; symbol Device:R -> LegacySymbols:R
- R3: footprint Resistor_SMD:R_0805_2012Metric -> LegacyBoard:R3_R_0805_2012Metric; symbol Device:R -> LegacySymbols:R
- R4: footprint Resistor_SMD:R_0805_2012Metric -> LegacyBoard:R4_R_0805_2012Metric; symbol Device:R -> LegacySymbols:R
- R5: footprint Resistor_SMD:R_0805_2012Metric -> LegacyBoard:R5_R_0805_2012Metric; symbol Device:R -> LegacySymbols:R
- R6: footprint Resistor_SMD:R_0805_2012Metric -> LegacyBoard:R6_R_0805_2012Metric; symbol Device:R -> LegacySymbols:R
- R7: footprint Resistor_SMD:R_0805_2012Metric -> LegacyBoard:R7_R_0805_2012Metric; symbol Device:R -> LegacySymbols:R
- R8: footprint Resistor_SMD:R_0805_2012Metric -> LegacyBoard:R8_R_0805_2012Metric; symbol Device:R -> LegacySymbols:R
- R9: footprint Resistor_SMD:R_0805_2012Metric -> LegacyBoard:R9_R_0805_2012Metric; symbol Device:R -> LegacySymbols:R
- SW1: footprint Button_Switch_SMD:SW_Push_1P1T_XKB_TS-1187A -> LegacyBoard:SW1_SW_Push_1P1T_XKB_TS-1187A; symbol Switch:SW_Push -> LegacySymbols:SW_Push
- SW2: footprint Button_Switch_SMD:SW_Push_1P1T_XKB_TS-1187A -> LegacyBoard:SW2_SW_Push_1P1T_XKB_TS-1187A; symbol Switch:SW_Push -> LegacySymbols:SW_Push
- TP1: footprint TestPoint:TestPoint_Pad_D2.0mm -> LegacyBoard:TP1_TestPoint_Pad_D2.0mm; symbol Connector:TestPoint -> LegacySymbols:TestPoint
- TP2: footprint TestPoint:TestPoint_Pad_D2.0mm -> LegacyBoard:TP2_TestPoint_Pad_D2.0mm; symbol Connector:TestPoint -> LegacySymbols:TestPoint
- TP3: footprint TestPoint:TestPoint_Pad_D2.0mm -> LegacyBoard:TP3_TestPoint_Pad_D2.0mm; symbol Connector:TestPoint -> LegacySymbols:TestPoint
- TP4: footprint TestPoint:TestPoint_Pad_D2.0mm -> LegacyBoard:TP4_TestPoint_Pad_D2.0mm; symbol Connector:TestPoint -> LegacySymbols:TestPoint
- TP5: footprint TestPoint:TestPoint_Pad_D2.0mm -> LegacyBoard:TP5_TestPoint_Pad_D2.0mm; symbol Connector:TestPoint -> LegacySymbols:TestPoint
- TP6: footprint TestPoint:TestPoint_Pad_D2.0mm -> LegacyBoard:TP6_TestPoint_Pad_D2.0mm; symbol Connector:TestPoint -> LegacySymbols:TestPoint
- TP7: footprint TestPoint:TestPoint_Pad_D2.0mm -> LegacyBoard:TP7_TestPoint_Pad_D2.0mm; symbol Connector:TestPoint -> LegacySymbols:TestPoint
- U1: footprint Package_TO_SOT_SMD:SOT-23 -> LegacyBoard:U1_SOT-23; symbol onionStraws:APX803L -> LegacySymbols:APX803L
- U2: footprint RF_Module:ESP32-C3-WROOM-02 -> LegacyBoard:U2_ESP32-C3-WROOM-02; symbol RF_Module:ESP32-C3-WROOM-02 -> LegacySymbols:ESP32-C3-WROOM-02
- U3: footprint Package_TO_SOT_SMD:TO-263-2 -> LegacyBoard:U3_TO-263-2; symbol Regulator_Linear:L7805 -> LegacySymbols:L7805
- U4: footprint Package_TO_SOT_SMD:SOT-23-6 -> LegacyBoard:U4_SOT-23-6; symbol 74xGxx:74LVC2G07 -> LegacySymbols:74LVC2G07
- U5: footprint Package_TO_SOT_SMD:SOT-23-6 -> LegacyBoard:U5_SOT-23-6; symbol onionStraws:74LVC2G07_3v3 -> LegacySymbols:74LVC2G07_3v3
- U6: footprint Package_TO_SOT_SMD:SOT-89-3 -> LegacyBoard:U6_SOT-89-3; symbol Regulator_Linear:AP2204R-3.3 -> LegacySymbols:AP2204R-3.3
Other:
- note added: "Input voltage / current not yet qualified"
- note added: "Inrush and load current not yet qualified"
- note added: "Intended polarity / inrush circuit Qualification pending"
- note added: "U1 DNP: existing boards boot-looped. R3 EN pull-up retained; qualification pending."
- note removed: "Peak of 1.5 amps w/o inrush"
- note removed: "Reverse polarity protection and inrush current limit"
- note removed: "VDC +9v to +16v"
- note removed: "Voltage Supervisor, Hold ESP reset for 150ms after power reaches 2.9V. Prevent brownout at boot."
