File: pcb/rev3c/design/GEA-Adapter-Rev3C.kicad_pcb (KiCad board)
At the start: 4 copper layers, 99 x 40 mm, 100 parts, among them J1 8P8C, J5 Socket_XIAO_A, J6 Socket_XIAO_B, Q3 CJ3407, Q4 CJ3407, Q5 MMBT3904, U10 TPS1H200AQDGNRQ1, U4 74LVC2G07, U5 74LVC2G07_3v3, U8 AP63205WU, U9 TPS1H200AQDGNRQ1

Commit message: fix(pcb): rate Rev3C input OR diodes for switch limit
Parts:
- D14, D15: value MBR0540-TP -> STPS140Z
Changed lines of the file:
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@@
 			)
 		)
-		(property "Value" "MBR0540-TP"
+		(property "Value" "STPS140Z"
 			(at 0 2.1 0)
 			(layer "F.Fab")
@@
 			)
 		)
-		(property "Datasheet" ""
+		(property "Datasheet" "https://www.st.com/resource/en/datasheet/stps140z.pdf"
 			(at 0 0 0)
 			(unlocked yes)
@@
 			)
 		)
-		(property "Description" ""
+		(property "Description" "40 V, 1 A Schottky rectifier, SOD-123; maximum junction 150 degC; LCSC C155662"
 			(at 0 0 0)
 			(unlocked yes)
@@
 			)
 		)
+		(property "LCSC" "C155662"
+			(at 0 0 0)
+			(layer "F.Fab")
+			(hide yes)
+			(effects (font (size 1.27 1.27) (thickness 0.15)))
+		)
+		(property "Manufacturer" "STMicroelectronics"
+			(at 0 0 0)
+			(layer "F.Fab")
+			(hide yes)
+			(effects (font (size 1.27 1.27) (thickness 0.15)))
+		)
+		(property "MPN" "STPS140Z"
+			(at 0 0 0)
+			(layer "F.Fab")
+			(hide yes)
+			(effects (font (size 1.27 1.27) (thickness 0.15)))
+		)
 	)
 	(footprint "Diode_SMD:Nexperia_CFP3_SOD-123W"
@@
 			)
 		)
-		(property "Value" "MBR0540-TP"
+		(property "Value" "STPS140Z"
 			(at 0 2.1 0)
 			(layer "F.Fab")
@@
 			)
 		)
-		(property "Datasheet" ""
+		(property "Datasheet" "https://www.st.com/resource/en/datasheet/stps140z.pdf"
 			(at 0 0 0)
 			(unlocked yes)
@@
 			)
 		)
-		(property "Description" ""
+		(property "Description" "40 V, 1 A Schottky rectifier, SOD-123; maximum junction 150 degC; LCSC C155662"
 			(at 0 0 0)
 			(unlocked yes)
@@
 			)
 		)
+		(property "LCSC" "C155662"
+			(at 0 0 0)
+			(layer "F.Fab")
+			(hide yes)
+			(effects (font (size 1.27 1.27) (thickness 0.15)))
+		)
+		(property "Manufacturer" "STMicroelectronics"
+			(at 0 0 0)
+			(layer "F.Fab")
+			(hide yes)
+			(effects (font (size 1.27 1.27) (thickness 0.15)))
+		)
+		(property "MPN" "STPS140Z"
+			(at 0 0 0)
+			(layer "F.Fab")
+			(hide yes)
+			(effects (font (size 1.27 1.27) (thickness 0.15)))
+		)
 	)
