File: pcb/rev3a/design/GEA-Adapter-Rev3A.kicad_pcb (KiCad board)
At the start: 4 copper layers, 88.7 x 40 mm, 115 parts, among them J1 8P8C, J2 RECOVERY, J4 USB_C_Receptacle_USB2.0_16P, Q3 CJ3407, Q4 CJ3407, Q5 MMBT3904, SW1 SW_Push, SW2 SW_Push, U10 TPS1H200AQDGNRQ1, U2 ESP32-C3-WROOM-02, U4 74LVC2G07, U5 74LVC2G07_3v3, U6 AP2112K-3.3, U7 USBLC6-2SC6, U8 AP63205WU, U9 TPS1H200AQDGNRQ1

Commit message: fix(pcb): backport Rev3A input diode rating repair
Parts:
- D14, D15: value MBR0540-TP -> STPS140Z
Changed lines of the file:
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@@
 			)
 		)
-		(property "Value" "MBR0540-TP"
+		(property "Value" "STPS140Z"
 			(at 0 2.1 0)
 			(layer "F.Fab")
@@
 			)
 		)
-		(property "Datasheet" ""
+		(property "Datasheet" "https://www.st.com/resource/en/datasheet/stps140z.pdf"
 			(at 0 0 0)
 			(unlocked yes)
@@
 			)
 		)
-		(property "Description" ""
+		(property "Description" "40 V, 1 A Schottky rectifier, SOD-123; maximum junction 150 degC; LCSC C155662"
 			(at 0 0 0)
 			(unlocked yes)
@@
 			)
 		)
+		(property "LCSC" "C155662"
+			(at 0 0 0)
+			(layer "F.Fab")
+			(hide yes)
+			(effects (font (size 1.27 1.27) (thickness 0.15)))
+		)
+		(property "Manufacturer" "STMicroelectronics"
+			(at 0 0 0)
+			(layer "F.Fab")
+			(hide yes)
+			(effects (font (size 1.27 1.27) (thickness 0.15)))
+		)
+		(property "MPN" "STPS140Z"
+			(at 0 0 0)
+			(layer "F.Fab")
+			(hide yes)
+			(effects (font (size 1.27 1.27) (thickness 0.15)))
+		)
 	)
 	(footprint "Diode_SMD:Nexperia_CFP3_SOD-123W"
@@
 			)
 		)
-		(property "Value" "MBR0540-TP"
+		(property "Value" "STPS140Z"
 			(at 0 2.1 0)
 			(layer "F.Fab")
@@
 			)
 		)
-		(property "Datasheet" ""
+		(property "Datasheet" "https://www.st.com/resource/en/datasheet/stps140z.pdf"
 			(at 0 0 0)
 			(unlocked yes)
@@
 			)
 		)
-		(property "Description" ""
+		(property "Description" "40 V, 1 A Schottky rectifier, SOD-123; maximum junction 150 degC; LCSC C155662"
 			(at 0 0 0)
 			(unlocked yes)
@@
 			)
 		)
+		(property "LCSC" "C155662"
+			(at 0 0 0)
+			(layer "F.Fab")
+			(hide yes)
+			(effects (font (size 1.27 1.27) (thickness 0.15)))
+		)
+		(property "Manufacturer" "STMicroelectronics"
+			(at 0 0 0)
+			(layer "F.Fab")
+			(hide yes)
+			(effects (font (size 1.27 1.27) (thickness 0.15)))
+		)
+		(property "MPN" "STPS140Z"
+			(at 0 0 0)
+			(layer "F.Fab")
+			(hide yes)
+			(effects (font (size 1.27 1.27) (thickness 0.15)))
+		)
 	)
